File: combined-pcb.sch (KiCad schematic (older format))
At the start: 11 parts, among them J1 CON_HEADER_1X02-PTH, J2 CON_HEADER_1X03-PTH, Q1 TRANSISTOR_NPNTO92, U1 ARDUINO_MINI, U2 NCP1117ST33T3G, U3 BLUETOOTH-HC05

Commit message: added kicad files
Parts:
- C1, C2: value CAPACITOR_NPOL-PTH_0.1\" -> C
- gave numbers to parts that had none: 1
Connections:
- net labels added: GND
Changed lines of the file:
@@
 P 1600 3750
 F 0 "C1" H 1700 3950 50  0000 L BNN
-F 1 "CAPACITOR_NPOL-PTH_0.1\"" H 1700 3850 50  0000 L BNN
+F 1 "C" H 1700 3850 50  0000 L BNN
 F 2 "dp_devices-C0.1PTH" H 1600 3900 50  0001 C CNN
 F 3 "" H 1600 3750 60  0000 C CNN
@@
 P 3050 3650
 F 0 "C2" H 3150 3850 50  0000 L BNN
-F 1 "CAPACITOR_NPOL-PTH_0.1\"" H 3150 3750 50  0000 L BNN
+F 1 "C" H 3150 3750 50  0000 L BNN
 F 2 "dp_devices-C0.1PTH" H 3050 3800 50  0001 C CNN
 F 3 "" H 3050 3650 60  0000 C CNN
@@
 	3050 3500 3350 3500
 $Comp
-L TRANSISTOR_NPNTO92 Q?
+L TRANSISTOR_NPNTO92 Q2
 U 1 1 53ADDBF4
 P 4200 3050
-F 0 "Q?" H 4350 3200 50  0000 L BNN
+F 0 "Q2" H 4350 3200 50  0000 L BNN
 F 1 "TRANSISTOR_NPNTO92" H 4350 2850 50  0000 L BNN
 F 2 "SparkFun-TO-92" H 4700 3050 50  0001 C CNN
@@
 Wire Wire Line
 	1350 6050 1500 6050
+Text Label 2800 4300 0    60   ~ 0
+GND
 $EndSCHEMATC
