File: mainboard/mainboard-pcb.sch (KiCad schematic (older format))
At the start: 18 parts, among them IC1 ATTINY2313-S, K1 CONN_3, P1 CONN_2, P2 CONN_5, P3 CONN_3X2, Q1 MOSFET_N, SW1 SW_PUSH, SW2 SW_PUSH, U1 NCP1117ST33T3G

Commit message: kicad file done
Parts:
- C1, C2, C3: footprint (none) -> SMD_Packages:SM0603_Capa
- D1: footprint (none) -> LEDs:LED-0805
- IC1: footprint SO20 -> SMD_Packages:SO20L
- K1: footprint (none) -> Pin_Headers:Pin_Header_Straight_1x03
- P1: footprint (none) -> Pin_Headers:Pin_Header_Straight_1x02
- P2: footprint (none) -> Pin_Headers:Pin_Header_Straight_1x05
- P3: footprint (none) -> Pin_Headers:Pin_Header_Straight_2x03
- Q1: footprint (none) -> SMD_Packages:SOT23
- R1, R2, R3, R4, R5: footprint (none) -> SMD_Packages:SM0603
- SW1, SW2: footprint (none) -> Discret:SW_PUSH
- U1: footprint (none) -> SMD_Packages:SOT223
Connections:
- net at IC1.1 (PA2(~RESET~/dW)), P3.5: now also R2.2
- net at C2.1, C3.1, IC1.20 (VCC)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: now also R2.1
Changed lines of the file:
@@
 LIBS:contrib
 LIBS:valves
+LIBS:mainboard-pcb-cache
 EELAYER 24 0
 EELAYER END
@@
 F 0 "IC1" H 3550 4250 40  0000 C CNN
 F 1 "ATTINY2313-S" H 5250 2350 40  0000 C CNN
-F 2 "SO20" H 4500 3250 35  0000 C CIN
+F 2 "SMD_Packages:SO20L" H 4500 3250 35  0000 C CIN
 F 3 "" H 4500 3250 60  0000 C CNN
 	1    4500 3250
@@
 F 0 "U1" H 1550 2300 40  0000 C CNN
 F 1 "NCP1117ST33T3G" H 1550 2250 40  0000 C CNN
-F 2 "" H 1550 2050 60  0000 C CNN
+F 2 "SMD_Packages:SOT223" H 1550 2050 60  0001 C CNN
 F 3 "" H 1550 2050 60  0000 C CNN
 	1    1550 2050
@@
 $EndComp
 $Comp
-L +BATT #PWR5
+L +BATT #PWR01
 U 1 1 53D27475
 P 2450 1250
-F 0 "#PWR5" H 2450 1200 20  0001 C CNN
+F 0 "#PWR01" H 2450 1200 20  0001 C CNN
 F 1 "+BATT" H 2450 1350 30  0000 C CNN
 F 2 "" H 2450 1250 60  0000 C CNN
@@
 $EndComp
 $Comp
-L GND #PWR4
+L GND #PWR02
 U 1 1 53D274A5
 P 2150 1200
-F 0 "#PWR4" H 2150 1200 30  0001 C CNN
+F 0 "#PWR02" H 2150 1200 30  0001 C CNN
 F 1 "GND" H 2150 1130 30  0001 C CNN
 F 2 "" H 2150 1200 60  0000 C CNN
@@
 F 0 "C1" H 800 2100 40  0000 L CNN
 F 1 "C" H 806 1915 40  0000 L CNN
-F 2 "" H 838 1850 30  0000 C CNN
+F 2 "SMD_Packages:SM0603_Capa" H 838 1850 30  0001 C CNN
 F 3 "" H 800 2000 60  0000 C CNN
 	1    800  2000
@@
 F 0 "C2" H 2300 2150 40  0000 L CNN
 F 1 "C" H 2306 1965 40  0000 L CNN
-F 2 "" H 2338 1900 30  0000 C CNN
+F 2 "SMD_Packages:SM0603_Capa" H 2338 1900 30  0001 C CNN
 F 3 "" H 2300 2050 60  0000 C CNN
 	1    2300 2050
@@
 F 0 "C3" H 4450 1700 40  0000 L CNN
 F 1 "C" H 4456 1515 40  0000 L CNN
-F 2 "" H 4488 1450 30  0000 C CNN
+F 2 "SMD_Packages:SM0603_Capa" H 4488 1450 30  0001 C CNN
 F 3 "" H 4450 1600 60  0000 C CNN
 	1    4450 1600
@@
 F 0 "P2" V 6800 2300 50  0000 C CNN
 F 1 "CONN_5" V 6900 2300 50  0000 C CNN
-F 2 "" H 6850 2300 60  0000 C CNN
+F 2 "Pin_Headers:Pin_Header_Straight_1x05" H 6850 2300 60  0001 C CNN
 F 3 "" H 6850 2300 60  0000 C CNN
 	1    6850 2300
@@
 F 0 "K1" V 1450 3800 50  0000 C CNN
 F 1 "CONN_3" V 1550 3800 40  0000 C CNN
-F 2 "" H 1500 3800 60  0000 C CNN
+F 2 "Pin_Headers:Pin_Header_Straight_1x03" H 1500 3800 60  0001 C CNN
 F 3 "" H 1500 3800 60  0000 C CNN
 	1    1500 3800
@@
 F 0 "SW1" H 4050 5810 50  0000 C CNN
 F 1 "SW_PUSH" H 3900 5620 50  0000 C CNN
-F 2 "" H 3900 5700 60  0000 C CNN
+F 2 "Discret:SW_PUSH" H 3900 5700 60  0001 C CNN
 F 3 "" H 3900 5700 60  0000 C CNN
 	1    3900 5700
@@
 F 0 "SW2" H 5300 5810 50  0000 C CNN
 F 1 "SW_PUSH" H 5150 5620 50  0000 C CNN
-F 2 "" H 5150 5700 60  0000 C CNN
+F 2 "Discret:SW_PUSH" H 5150 5700 60  0001 C CNN
 F 3 "" H 5150 5700 60  0000 C CNN
 	1    5150 5700
@@
 F 0 "D1" H 2050 5650 50  0000 C CNN
 F 1 "LED" H 2050 5450 50  0000 C CNN
-F 2 "" H 2050 5550 60  0000 C CNN
+F 2 "LEDs:LED-0805" H 2050 5550 60  0001 C CNN
 F 3 "" H 2050 5550 60  0000 C CNN
 	1    2050 5550
@@
 F 0 "R1" V 2780 5550 40  0000 C CNN
 F 1 "R" V 2707 5551 40  0000 C CNN
-F 2 "" V 2630 5550 30  0000 C CNN
+F 2 "SMD_Packages:SM0603" V 2630 5550 30  0001 C CNN
 F 3 "" H 2700 5550 30  0000 C CNN
 	1    2700 5550
@@
 F 0 "R5" V 6680 3700 40  0000 C CNN
 F 1 "R" V 6607 3701 40  0000 C CNN
-F 2 "" V 6530 3700 30  0000 C CNN
+F 2 "SMD_Packages:SM0603" V 6530 3700 30  0001 C CNN
 F 3 "" H 6600 3700 30  0000 C CNN
 	1    6600 3700
@@
 F 0 "R3" V 3730 1150 40  0000 C CNN
 F 1 "R" V 3657 1151 40  0000 C CNN
-F 2 "" V 3580 1150 30  0000 C CNN
+F 2 "SMD_Packages:SM0603" V 3580 1150 30  0001 C CNN
 F 3 "" H 3650 1150 30  0000 C CNN
 	1    3650 1150
@@
 F 0 "R4" V 4230 950 40  0000 C CNN
 F 1 "R" V 4157 951 40  0000 C CNN
-F 2 "" V 4080 950 30  0000 C CNN
+F 2 "SMD_Packages:SM0603" V 4080 950 30  0001 C CNN
 F 3 "" H 4150 950 30  0000 C CNN
 	1    4150 950
@@
 F 0 "Q1" H 2460 4270 60  0000 R CNN
 F 1 "MOSFET_N" H 2460 3950 60  0000 R CNN
-F 2 "" H 2450 4100 60  0000 C CNN
+F 2 "SMD_Packages:SOT23" H 2450 4100 60  0001 C CNN
 F 3 "" H 2450 4100 60  0000 C CNN
 	1    2450 4100
@@
 F 0 "P1" V 1100 900 40  0000 C CNN
 F 1 "CONN_2" V 1200 900 40  0000 C CNN
-F 2 "" H 1150 900 60  0000 C CNN
+F 2 "Pin_Headers:Pin_Header_Straight_1x02" H 1150 900 60  0001 C CNN
 F 3 "" H 1150 900 60  0000 C CNN
 	1    1150 900
@@
 	1500 1250 1250 1250
 $Comp
-L GND #PWR2
+L GND #PWR03
 U 1 1 53D28115
 P 1550 2450
-F 0 "#PWR2" H 1550 2450 30  0001 C CNN
+F 0 "#PWR03" H 1550 2450 30  0001 C CNN
 F 1 "GND" H 1550 2380 30  0001 C CNN
 F 2 "" H 1550 2450 60  0000 C CNN
@@
 $EndComp
 $Comp
-L GND #PWR8
+L GND #PWR04
 U 1 1 53D281B9
 P 4500 4500
-F 0 "#PWR8" H 4500 4500 30  0001 C CNN
+F 0 "#PWR04" H 4500 4500 30  0001 C CNN
 F 1 "GND" H 4500 4430 30  0001 C CNN
 F 2 "" H 4500 4500 60  0000 C CNN
@@
 $EndComp
 $Comp
-L GND #PWR10
+L GND #PWR05
 U 1 1 53D2825D
 P 6250 1950
-F 0 "#PWR10" H 6250 1950 30  0001 C CNN
+F 0 "#PWR05" H 6250 1950 30  0001 C CNN
 F 1 "GND" H 6250 1880 30  0001 C CNN
 F 2 "" H 6250 1950 60  0000 C CNN
@@
 $EndComp
 $Comp
-L GND #PWR7
+L GND #PWR06
 U 1 1 53D28381
 P 3950 6200
-F 0 "#PWR7" H 3950 6200 30  0001 C CNN
+F 0 "#PWR06" H 3950 6200 30  0001 C CNN
 F 1 "GND" H 3950 6130 30  0001 C CNN
 F 2 "" H 3950 6200 60  0000 C CNN
@@
 $EndComp
 $Comp
-L GND #PWR9
+L GND #PWR07
 U 1 1 53D283B5
 P 5100 6200
-F 0 "#PWR9" H 5100 6200 30  0001 C CNN
+F 0 "#PWR07" H 5100 6200 30  0001 C CNN
 F 1 "GND" H 5100 6130 30  0001 C CNN
 F 2 "" H 5100 6200 60  0000 C CNN
@@
 $EndComp
 $Comp
-L GND #PWR6
+L GND #PWR08
 U 1 1 53D28409
 P 2750 6250
-F 0 "#PWR6" H 2750 6250 30  0001 C CNN
+F 0 "#PWR08" H 2750 6250 30  0001 C CNN
 F 1 "GND" H 2750 6180 30  0001 C CNN
 F 2 "" H 2750 6250 60  0000 C CNN
@@
 $EndComp
 $Comp
-L GND #PWR1
+L GND #PWR09
 U 1 1 53D2849D
 P 1350 3400
-F 0 "#PWR1" H 1350 3400 30  0001 C CNN
+F 0 "#PWR09" H 1350 3400 30  0001 C CNN
 F 1 "GND" H 1350 3330 30  0001 C CNN
 F 2 "" H 1350 3400 60  0000 C CNN
@@
 F 0 "R2" V 3630 2100 40  0000 C CNN
 F 1 "R" V 3557 2101 40  0000 C CNN
-F 2 "" V 3480 2100 30  0000 C CNN
+F 2 "SMD_Packages:SM0603" V 3480 2100 30  0001 C CNN
 F 3 "" H 3550 2100 30  0000 C CNN
 	1    3550 2100
@@
 $EndComp
 Wire Wire Line
-	3800 2100 4500 2100
-Wire Wire Line
 	4500 2000 4500 2150
-Wire Wire Line
-	3300 2100 3300 2450
 Wire Wire Line
 	1850 2450 3350 2450
@@
 F 0 "P3" H 1100 6850 50  0000 C CNN
 F 1 "CONN_3X2" V 1100 6650 40  0000 C CNN
-F 2 "" H 1100 6600 60  0000 C CNN
+F 2 "Pin_Headers:Pin_Header_Straight_2x03" H 1100 6600 60  0001 C CNN
 F 3 "" H 1100 6600 60  0000 C CNN
 	1    1100 6600
@@
 	3150 2000 4500 2000
 $Comp
-L GND #PWR3
+L GND #PWR010
 U 1 1 53D2B838
 P 1550 6900
-F 0 "#PWR3" H 1550 6900 30  0001 C CNN
+F 0 "#PWR010" H 1550 6900 30  0001 C CNN
 F 1 "GND" H 1550 6830 30  0001 C CNN
 F 2 "" H 1550 6900 60  0000 C CNN
@@
 Wire Wire Line
 	1550 6650 1550 6900
+Wire Wire Line
+	3800 2100 4500 2100
+Connection ~ 4500 2100
+Wire Wire Line
+	3350 2450 3350 2300
+Wire Wire Line
+	3350 2300 3250 2300
+Wire Wire Line
+	3250 2300 3250 2100
+Wire Wire Line
+	3250 2100 3300 2100
 $EndSCHEMATC
